File: design_files/AST1003.sch (EAGLE design)
At the start: 12 parts, among them J1 SM05B, U2 ATTINY841

Commit message: updated documentation
Parts:
- C3: value 10uF -> 1uF; device tinycircuits:AS-ITM-00002 -> tinycircuits:AS-ITM-00410; PARTNO (none) -> AS-ITM-00410; VALUE (none) -> 1uF
- R2: value 0.0 -> 1.00K; device tinycircuits:AS-ITM-00076 -> tinycircuits:AS-ITM-00003; PARTNO (none) -> AS-ITM-00003; VALUE (none) -> 1.00K
Other:
- note added: "2"
- note added: "Wireling Cap Touch"
- note removed: "1"
- note removed: "Cap. Touch Slider Board"
Changed lines of the file:
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@@
 <layer number="59" name="Invisible" color="7" fill="1" visible="no" active="no"/>
 <layer number="61" name="stand" color="7" fill="1" visible="no" active="no"/>
+<layer number="88" name="SimResults" color="9" fill="1" visible="yes" active="yes"/>
+<layer number="89" name="SimProbes" color="9" fill="1" visible="yes" active="yes"/>
 <layer number="90" name="Modules" color="5" fill="1" visible="yes" active="yes"/>
 <layer number="91" name="Nets" color="2" fill="1" visible="yes" active="yes"/>
@@
 <layer number="158" name="bResistor" color="7" fill="1" visible="no" active="yes"/>
 <layer number="159" name="henwayCAP" color="13" fill="1" visible="yes" active="yes"/>
+<layer number="160" name="IDFDebug" color="7" fill="1" visible="yes" active="yes"/>
 <layer number="191" name="mNets" color="7" fill="1" visible="yes" active="yes"/>
 <layer number="192" name="mBusses" color="7" fill="1" visible="yes" active="yes"/>
@@
 <part name="P+3" library="tinycircuits" deviceset="VCC" device=""/>
 <part name="GND1" library="tinycircuits" deviceset="GND" device=""/>
-<part name="C3" library="tinycircuits" deviceset="AS-ITM-00002" device="" value="10uF"/>
+<part name="C3" library="tinycircuits" deviceset="AS-ITM-00410" device="" value="1uF">
+<attribute name="PARTNO" value="AS-ITM-00410"/>
+<attribute name="VALUE" value="1uF"/>
+</part>
 <part name="P+5" library="tinycircuits" deviceset="VCC" device=""/>
 <part name="GND4" library="tinycircuits" deviceset="GND" device=""/>
-<part name="R2" library="tinycircuits" deviceset="AS-ITM-00076" device="" value="0.0"/>
+<part name="R2" library="tinycircuits" deviceset="AS-ITM-00003" device="" value="1.00K">
+<attribute name="PARTNO" value="AS-ITM-00003"/>
+<attribute name="VALUE" value="1.00K"/>
+</part>
 </parts>
 <sheets>
 <sheet>
 <plain>
-<text x="340.868" y="17.272" size="3.556" layer="94" font="vector">Cap. Touch Slider Board</text>
+<text x="340.868" y="17.272" size="3.556" layer="94" font="vector">Wireling Cap Touch</text>
 <text x="327.152" y="6.35" size="3.556" layer="94" font="vector">AS-SCH-AST1003</text>
-<text x="416.56" y="6.858" size="3.556" layer="94" font="vector">1</text>
+<text x="416.56" y="6.858" size="3.556" layer="94" font="vector">2</text>
 <text x="165.1" y="185.42" size="5.08" layer="94" font="vector">Capacitive Touch Slider</text>
 <text x="45.72" y="35.56" size="3.048" layer="91">Released under the Creative Commons Attribution Share-Alike 3.0 License</text>
